File: stm32_reference_project.sch (KiCad schematic (older format))
At the start: 42 parts, among them J1 USB_Serial, J2 PROG_HDR, SW1 RESET, SW2 BAT_SELECT, SW3 BOOT_SELECT, U1 MIC5504-3.3YM5, U2 STM32F103C8Tx, Y1 8Mhz, Y2 32.768K

Commit message: DIP switches won't fly, use a header for it
Parts:
- removed R6, R9: 10k, Resistor_SMD:R_0603_1608Metric, symbol Device:R
- removed SW3: BOOT_SELECT, Button_Switch_THT:SW_DIP_SPSTx02_Slide_9.78x7.26mm_W7.62mm_P2.54mm, symbol Switch:SW_DPDT_x2
- added J?: BOOT_SELECT, Connector:Tag-Connect_TC2030-IDC-FP_2x03_P1.27mm_Vertical, symbol Connector_Generic:Conn_02x03_Odd_Even
- added R? (x2): 10k, Resistor_SMD:R_0603_1608Metric, symbol Device:R
Connections:
- wire segments 182 -> 188
Other:
- note added: "The boot header is present for development when\ncomplete the off positions can be soldered\ntogether to save the cost of the header\n\nBOOT_SELECT:\nUser Flash (Normal): BOOT0-X, BOOT1-Off\nSystem Memory: BOOT0-Off, BOOT1-On\nEmbedded SRAM: BOOT0-On, BOOT1-On"
- note added: "This LED matches the expectation of the\nstm32duino bootloader "generic_boot20_pc13.bin"\nin the event I want to use that for firmware\ndevelopment"
- note added: "Vbat can be powered by a seperate battery to keep the\nRTC and backup registers running when main power is\nremoved, otherwise it should be connected to the main\nsupply with this decoupling cap."
- note added: "Vdd / Vdda require a voltage of\n2.0V - 3.6V (2.4V - 3.6V when the ADC is used)\nVbat requires a voltage of 1.8V - 3.6V"
- note removed: "BOOT_SELECT:\nUser Flash (Normal): BOOT0-X, BOOT1-Off\nSystem Memory (Prog via USART1): BOOT0-Off, BOOT1-On\nEmbedded SRAM: BOOT0-On, BOOT1-On"
- note removed: "This matches the expectation of the normal\narduino stm32 bootloader"
- note removed: "Vbat can be powered by a seperate battery to keep the\nRTC and backup registers running when main power is\nremoved, otherwise it should be connected to the main\nsupply with a decoupling cap.\n\nIn real applications one of these two options should be\nselected."
- note removed: "Vdd, and Vdda require a voltage of\n2.0V - 3.6V (2.4V - 3.6V when the ADC is used)\n\nVbat requires a voltage of 1.8V - 3.6V"
- moved on the sheet: C17, C18, D3, D4, FB1, R7, R8

Commit message: Some parts weren't labelled
Parts:
- gave numbers to parts that had none: 3
- renumbered C13 to C12, C12 to C13, C16 to C15, C15 to C16, R7 to R6
Changed lines of the file:
@@
 $EndComp
 $Comp
-L power:GND #PWR025
+L power:GND #PWR026
 U 1 1 5C8448B4
 P 9900 4800
-F 0 "#PWR025" H 9900 4550 50  0001 C CNN
+F 0 "#PWR026" H 9900 4550 50  0001 C CNN
 F 1 "GND" H 9905 4627 50  0000 C CNN
 F 2 "" H 9900 4800 50  0001 C CNN
@@
 $EndComp
 $Comp
-L power:VDD #PWR024
+L power:VDD #PWR025
 U 1 1 5C8A198A
 P 9900 3800
-F 0 "#PWR024" H 9900 3650 50  0001 C CNN
+F 0 "#PWR025" H 9900 3650 50  0001 C CNN
 F 1 "VDD" H 9917 3973 50  0000 C CNN
 F 2 "" H 9900 3800 50  0001 C CNN
@@
 $EndComp
 $Comp
-L Device:C C16
+L Device:C C15
 U 1 1 5C9F7C35
 P 4950 2150
-F 0 "C16" H 5065 2196 50  0000 L CNN
+F 0 "C15" H 5065 2196 50  0000 L CNN
 F 1 "1uF" H 5065 2105 50  0000 L CNN
 F 2 "Capacitor_SMD:C_0603_1608Metric" H 4988 2000 50  0001 C CNN
@@
 	4650 6150 4650 6000
 $Comp
-L Device:C C15
+L Device:C C16
 U 1 1 5C7F9FBF
 P 4950 6150
-F 0 "C15" V 5200 6100 50  0000 L CNN
+F 0 "C16" V 5200 6100 50  0000 L CNN
 F 1 "0.1uF" V 5100 6050 50  0000 L CNN
 F 2 "Capacitor_SMD:C_0603_1608Metric" H 4988 6000 50  0001 C CNN
@@
 USB_VCC
 $Comp
-L Device:C C12
+L Device:C C13
 U 1 1 5C5EAB9E
 P 3700 2150
-F 0 "C12" H 3815 2196 50  0000 L CNN
+F 0 "C13" H 3815 2196 50  0000 L CNN
 F 1 "1uF" H 3815 2105 50  0000 L CNN
 F 2 "Capacitor_SMD:C_0603_1608Metric" H 3738 2000 50  0001 C CNN
@@
 Connection ~ 1600 6500
 $Comp
-L Device:R R7
+L Device:R R6
 U 1 1 5D04195A
 P 7900 5950
-F 0 "R7" V 7693 5950 50  0000 C CNN
+F 0 "R6" V 7693 5950 50  0000 C CNN
 F 1 "390" V 7784 5950 50  0000 C CNN
 F 2 "Resistor_SMD:R_0603_1608Metric" V 7830 5950 50  0001 C CNN
@@
 $EndComp
 $Comp
-L power:GND #PWR028
+L power:GND #PWR022
 U 1 1 5D042D15
 P 8650 6100
-F 0 "#PWR028" H 8650 5850 50  0001 C CNN
+F 0 "#PWR022" H 8650 5850 50  0001 C CNN
 F 1 "GND" H 8655 5927 50  0000 C CNN
 F 2 "" H 8650 6100 50  0001 C CNN
@@
 $EndComp
 $Comp
-L power:GND #PWR029
+L power:GND #PWR027
 U 1 1 5D0447BF
 P 10500 6100
-F 0 "#PWR029" H 10500 5850 50  0001 C CNN
+F 0 "#PWR027" H 10500 5850 50  0001 C CNN
 F 1 "GND" H 10505 5927 50  0000 C CNN
 F 2 "" H 10500 6100 50  0001 C CNN
@@
 $EndComp
 $Comp
-L Device:C C13
+L Device:C C12
 U 1 1 5C7AE180
 P 3500 5250
-F 0 "C13" H 3615 5296 50  0000 L CNN
+F 0 "C12" H 3615 5296 50  0000 L CNN
 F 1 "10uF" H 3615 5205 50  0000 L CNN
 F 2 "Capacitor_SMD:C_0603_1608Metric" H 3538 5100 50  0001 C CNN
@@
 BOOT0
 $Comp
-L Device:R R?
+L Device:R R9
 U 1 1 5D0701C5
 P 10050 2400
-AR Path="/5D0701C5" Ref="R?"  Part="1"
+AR Path="/5D0701C5" Ref="R9"  Part="1"
 AR Path="/5C77D6A4/5D0701C5" Ref="R?"  Part="1"
-F 0 "R?" V 9843 2400 50  0000 C CNN
+F 0 "R9" V 9843 2400 50  0000 C CNN
 F 1 "10k" V 9934 2400 50  0000 C CNN
 F 2 "Resistor_SMD:R_0603_1608Metric" V 9980 2400 50  0001 C CNN
@@
 	9900 2100 9900 2300
 $Comp
-L Device:R R?
+L Device:R R7
 U 1 1 5D0701C6
 P 9050 2400
-AR Path="/5D0701C6" Ref="R?"  Part="1"
+AR Path="/5D0701C6" Ref="R7"  Part="1"
 AR Path="/5C77D6A4/5D0701C6" Ref="R?"  Part="1"
-F 0 "R?" V 8843 2400 50  0000 C CNN
+F 0 "R7" V 8843 2400 50  0000 C CNN
 F 1 "10k" V 8934 2400 50  0000 C CNN
 F 2 "Resistor_SMD:R_0603_1608Metric" V 8980 2400 50  0001 C CNN
@@
 	10200 2400 10500 2400
 $Comp
-L power:GND #PWR?
+L power:GND #PWR024
 U 1 1 5D0701C7
 P 9550 2800
-AR Path="/5D0701C7" Ref="#PWR?"  Part="1"
+AR Path="/5D0701C7" Ref="#PWR024"  Part="1"
 AR Path="/5C77D6A4/5D0701C7" Ref="#PWR?"  Part="1"
-F 0 "#PWR?" H 9550 2550 50  0001 C CNN
+F 0 "#PWR024" H 9550 2550 50  0001 C CNN
 F 1 "GND" H 9555 2627 50  0000 C CNN
 F 2 "" H 9550 2800 50  0001 C CNN
@@
 	9550 2800 9550 2700
 $Comp
-L power:VDD #PWR?
+L power:VDD #PWR023
 U 1 1 5D0701C8
 P 9550 2000
-F 0 "#PWR?" H 9550 1850 50  0001 C CNN
+F 0 "#PWR023" H 9550 1850 50  0001 C CNN
 F 1 "VDD" H 9567 2173 50  0000 C CNN
 F 2 "" H 9550 2000 50  0001 C CNN
@@
 P 9500 2400
 AR Path="/5C77D6A4/5D0701C9" Ref="J?"  Part="1"
-AR Path="/5D0701C9" Ref="J?"  Part="1"
-F 0 "J?" H 9500 2600 50  0000 L CNN
+AR Path="/5D0701C9" Ref="J3"  Part="1"
+F 0 "J3" H 9500 2600 50  0000 L CNN
 F 1 "BOOT_SELECT" H 9300 2200 50  0000 L CNN
 F 2 "Connector:Tag-Connect_TC2030-IDC-FP_2x03_P1.27mm_Vertical" H 9500 2400 50  0001 C CNN
